File: Circuit/PCB_JST/Lemmingometre_JST.kicad_pcb (KiCad board)
At the start: 2 copper layers, 30.6 x 77.6 mm, 16 parts

Commit message: Add Gerber files
Routing:
- net Net-(H2-Pin_3): track 18.3 -> 19.7 mm
- net Net-(MCU1-~{RST}): track 48.4 -> 49.0 mm
