File: Circuit/PCB_JST/Lemmingometre_JST.kicad_sch (KiCad schematic)
At the start: 15 parts

Commit message: Add Gerber files
Parts:
- removed H6: Conn_IR, Connector_JST:JST_PH_B3B-PH-K_1x03_P2.00mm_Vertical, symbol Connector:Conn_01x03_Pin
- added H4: Conn_PIR3, Connector_JST:JST_PH_B4B-PH-K_1x04_P2.00mm_Vertical, symbol Connector:Conn_01x04_Pin
- R1, R2: value R -> 1k
- R3, R4: value 5k -> 1M
- renumbered H4 to H2, H5 to H3
Connections:
- net at H1.1 (Pin_1), H2.1 (Pin_1), H3.1 (Pin_1)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: now also H4.1 (Pin_1)
- net at H1.2 (Pin_2), H2.2 (Pin_2), H3.2 (Pin_2)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: now also H4.2 (Pin_2)
- net at MCU1.11 (D4): now also H4.3 (Pin_3)
- net at MCU1.3 (D0): now also H4.4 (Pin_4)
- no-connect marks 7 -> 6
Changed lines of the file:
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@@
   (junction (at 180.34 114.3) (diameter 0) (color 0 0 0 0)
   )
+  (junction (at 176.53 80.01) (diameter 0) (color 0 0 0 0)
+  )
   (junction (at 156.21 68.58) (diameter 0) (color 0 0 0 0)
   )
-  (junction (at 172.72 80.01) (diameter 0) (color 0 0 0 0)
-  )
   (junction (at 110.49 82.55) (diameter 0) (color 0 0 0 0)
   )
   (junction (at 156.21 80.01) (diameter 0) (color 0 0 0 0)
   )
+  (junction (at 158.75 74.93) (diameter 0) (color 0 0 0 0)
+  )
   (junction (at 87.63 82.55) (diameter 0) (color 0 0 0 0)
   )
@@
   )
   (junction (at 184.15 109.22) (diameter 0) (color 0 0 0 0)
-  )
-  (junction (at 158.75 74.93) (diameter 0) (color 0 0 0 0)
   )
   (junction (at 153.67 123.19) (diameter 0) (color 0 0 0 0)
@@
   (no_connect (at 143.51 100.33))
   (no_connect (at 189.23 124.46))
-  (no_connect (at 163.83 90.17))
   (no_connect (at 151.13 80.01))
   (no_connect (at 143.51 97.79))
@@
     (stroke (width 0) (type default))
   )
+  (wire (pts (xy 176.53 73.66) (xy 176.53 80.01))
+    (stroke (width 0) (type default))
+  )
   (wire (pts (xy 107.95 99.06) (xy 111.76 99.06))
     (stroke (width 0) (type default))
@@
     (stroke (width 0) (type default))
   )
-  (wire (pts (xy 156.21 80.01) (xy 172.72 80.01))
+  (wire (pts (xy 158.75 74.93) (xy 179.07 74.93))
+    (stroke (width 0) (type default))
+  )
+  (wire (pts (xy 156.21 80.01) (xy 176.53 80.01))
     (stroke (width 0) (type default))
   )
@@
     (stroke (width 0) (type default))
   )
+  (wire (pts (xy 179.07 73.66) (xy 179.07 74.93))
+    (stroke (width 0) (type default))
+  )
   (wire (pts (xy 135.89 127) (xy 153.67 127))
     (stroke (width 0) (type default))
@@
     (stroke (width 0) (type default))
   )
-  (wire (pts (xy 175.26 74.93) (xy 158.75 74.93))
-    (stroke (width 0) (type default))
-  )
   (wire (pts (xy 189.23 121.92) (xy 171.45 121.92))
     (stroke (width 0) (type default))
@@
     (stroke (width 0) (type default))
   )
-  (wire (pts (xy 172.72 73.66) (xy 172.72 80.01))
-    (stroke (width 0) (type default))
-  )
   (wire (pts (xy 111.76 99.06) (xy 111.76 109.22))
     (stroke (width 0) (type default))
@@
     (stroke (width 0) (type default))
   )
+  (wire (pts (xy 173.99 86.36) (xy 173.99 73.66))
+    (stroke (width 0) (type default))
+  )
   (wire (pts (xy 158.75 74.93) (xy 135.89 74.93))
     (stroke (width 0) (type default))
   )
+  (wire (pts (xy 163.83 90.17) (xy 167.64 90.17))
+    (stroke (width 0) (type default))
+  )
   (wire (pts (xy 158.75 64.77) (xy 158.75 74.93))
     (stroke (width 0) (type default))
@@
     (stroke (width 0) (type default))
   )
+  (wire (pts (xy 170.18 100.33) (xy 170.18 86.36))
+    (stroke (width 0) (type default))
+  )
   (wire (pts (xy 180.34 114.3) (xy 180.34 127))
     (stroke (width 0) (type default))
@@
     (stroke (width 0) (type default))
   )
-  (wire (pts (xy 170.18 73.66) (xy 170.18 100.33))
-    (stroke (width 0) (type default))
-  )
   (wire (pts (xy 187.96 100.33) (xy 180.34 100.33))
     (stroke (width 0) (type default))
   )
+  (wire (pts (xy 176.53 80.01) (xy 205.74 80.01))
+    (stroke (width 0) (type default))
+  )
+  (wire (pts (xy 171.45 77.47) (xy 171.45 73.66))
+    (stroke (width 0) (type default))
+  )
   (wire (pts (xy 99.06 82.55) (xy 100.33 82.55))
     (stroke (width 0) (type default))
@@
     (stroke (width 0) (type default))
   )
+  (wire (pts (xy 167.64 90.17) (xy 167.64 77.47))
+    (stroke (width 0) (type default))
+  )
   (wire (pts (xy 153.67 120.65) (xy 153.67 123.19))
     (stroke (width 0) (type default))
   )
-  (wire (pts (xy 172.72 80.01) (xy 205.74 80.01))
-    (stroke (width 0) (type default))
-  )
   (wire (pts (xy 110.49 82.55) (xy 110.49 90.17))
     (stroke (width 0) (type default))
@@
     (stroke (width 0) (type default))
   )
-  (wire (pts (xy 175.26 73.66) (xy 175.26 74.93))
-    (stroke (width 0) (type default))
-  )
   (wire (pts (xy 156.21 68.58) (xy 156.21 80.01))
     (stroke (width 0) (type default))
@@
     (stroke (width 0) (type default))
   )
+  (wire (pts (xy 170.18 86.36) (xy 173.99 86.36))
+    (stroke (width 0) (type default))
+  )
   (wire (pts (xy 82.55 99.06) (xy 87.63 99.06))
     (stroke (width 0) (type default))
   )
   (wire (pts (xy 153.67 123.19) (xy 153.67 127))
+    (stroke (width 0) (type default))
+  )
+  (wire (pts (xy 167.64 77.47) (xy 171.45 77.47))
     (stroke (width 0) (type default))
   )
@@
   (symbol (lib_id "Connector:Conn_01x03_Pin") (at 77.47 99.06 0) (unit 1)
     (in_bom yes) (on_board yes) (dnp no)
-    (property "Reference" "H5" (at 76.2 91.44 0)
+    (property "Reference" "H3" (at 76.2 91.44 0)
       (effects (font (size 1.27 1.27)))
     )
@@
       (project "Lemmingometre_v2"
         (path "/1a876431-a50c-42b9-9211-97f8b75d64c0"
-          (reference "H5") (unit 1)
+          (reference "H3") (unit 1)
         )
       )
@@
       (effects (font (size 1.27 1.27)))
     )
-    (property "Value" "R" (at 104.14 95.25 90)
+    (property "Value" "1k" (at 104.14 95.25 90)
       (effects (font (size 1.27 1.27)))
     )
@@
       (effects (font (size 1.27 1.27)))
     )
-    (property "Value" "5k" (at 114.3 87.63 90)
+    (property "Value" "1M" (at 114.3 87.63 90)
       (effects (font (size 1.27 1.27)))
     )
@@
       (effects (font (size 1.27 1.27)))
     )
-    (property "Value" "R" (at 104.14 80.01 90)
+    (property "Value" "1k" (at 104.14 80.01 90)
       (effects (font (size 1.27 1.27)))
     )
@@
   (symbol (lib_id "Connector:Conn_01x03_Pin") (at 77.47 82.55 0) (unit 1)
     (in_bom yes) (on_board yes) (dnp no) (fields_autoplaced)
-    (property "Reference" "H4" (at 78.105 74.93 0)
+    (property "Reference" "H2" (at 78.105 74.93 0)
       (effects (font (size 1.27 1.27)))
     )
@@
       (project "Lemmingometre_v2"
         (path "/1a876431-a50c-42b9-9211-97f8b75d64c0"
-          (reference "H4") (unit 1)
+          (reference "H2") (unit 1)
         )
       )
@@
       (effects (font (size 1.27 1.27)))
     )
-    (property "Value" "5k" (at 115.57 106.68 90)
+    (property "Value" "1M" (at 115.57 106.68 90)
       (effects (font (size 1.27 1.27)))
     )
@@
     )
   )
+  (symbol (lib_id "Connector:Conn_01x04_Pin") (at 176.53 68.58 270) (unit 1)
+    (in_bom yes) (on_board yes) (dnp no) (fields_autoplaced)
+    (property "Reference" "H4" (at 175.26 63.5 90)
+      (effects (font (size 1.27 1.27)))
+    )
+    (property "Value" "Conn_PIR3" (at 175.26 66.04 90)
+      (effects (font (size 1.27 1.27)))
+    )
+    (property "Footprint" "Connector_JST:JST_PH_B4B-PH-K_1x04_P2.00mm_Vertical" (at 176.53 68.58 0)
+      (effects (font (size 1.27 1.27)) hide)
+    )
+    (property "Datasheet" "~" (at 176.53 68.58 0)
+      (effects (font (size 1.27 1.27)) hide)
+    )
+    (pin "1")
+    (pin "2")
+    (pin "3")
+    (pin "4")
+    (instances
+      (project "Lemmingometre_v2"
+        (path "/1a876431-a50c-42b9-9211-97f8b75d64c0"
+          (reference "H4") (unit 1)
+        )
+      )
+    )
+  )
   (symbol (lib_id "Connector:Conn_01x02_Pin") (at 158.75 59.69 270) (unit 1)
     (in_bom yes) (on_board yes) (dnp no) (fields_autoplaced)
@@
         )
       )
-    )
-  )
-  (symbol (lib_id "Connector:Conn_01x03_Pin") (at 172.72 68.58 270) (unit 1)
-    (in_bom yes) (on_board yes) (dnp no)
-    (property "Reference" "H6" (at 172.72 64.77 90)
-      (effects (font (size 1.27 1.27)))
-    )
-    (property "Value" "Conn_IR" (at 172.72 66.04 90)
-      (effects (font (size 1.27 1.27)))
-    )
-    (property "Footprint" "Connector_JST:JST_PH_B3B-PH-K_1x03_P2.00mm_Vertical" (at 172.72 68.58 0)
-      (effects (font (size 1.27 1.27)) hide)
-    )
-    (property "Datasheet" "~" (at 172.72 68.58 0)
-      (effects (font (size 1.27 1.27)) hide)
-    )
-    (pin "1")
-    (pin "2")
-    (pin "3")
-    (instances
-      (project "Lemmingometre_v2"
-        (path "/1a876431-a50c-42b9-9211-97f8b75d64c0"
-          (reference "H6") (unit 1)
-        )
-      )
